Commit message: 修改first_robot.urdf.xacro文件中参数为被正确使用的问题

File: chapt6/chapt_ws/src/fishbot_description/urdf/first_robot.urdf.xacro (robot description, xacro)
@@ -6,5 +6,5 @@
                 <origin xyz="0.0 0.0 0.0" rpy="0.0 0.0 0.0"/>
                 <geometry>
-                    <cylinder radius="0.1" length="0.12"/>
+                    <cylinder radius="${radius}" length="${length}"/>
                 </geometry>
                 <material name="white">
