Commit message: 添加机器人轮子，并添加一个空部件作为base_link的基座，以便选为原点，使得整体的位置处于地面以上

File: chapt6/chapt_ws/src/fishbot_description/urdf/fishbot/base.urdf.xacro (robot description, xacro)
@@ -13,4 +13,10 @@
             </visual>
         </link>
+        <link name="base_footprint" />
+        <joint name="base_joint" type="fixed">
+            <parent link="base_footprint"/>
+            <child link="base_link"/>
+            <origin xyz="0 0 ${length/2.0+0.032-0.001}" rpy="0.0 0.0 0.0"/>
+        </joint>
     </xacro:macro>
 </robot>

File: chapt6/chapt_ws/src/fishbot_description/urdf/fishbot/fishbot.urdf.xacro (robot description, xacro)
@@ -5,7 +5,13 @@
     <xacro:include filename="$(find fishbot_description)/urdf/fishbot/sensor/camera.urdf.xacro"/>
     <xacro:include filename="$(find fishbot_description)/urdf/fishbot/sensor/laser.urdf.xacro"/>
+    <xacro:include filename="$(find fishbot_description)/urdf/fishbot/actuator/wheel.urdf.xacro"/>
+    <xacro:include filename="$(find fishbot_description)/urdf/fishbot/actuator/caster.urdf.xacro"/>
     <xacro:base_xacro length="0.12" radius="0.1" />
     <xacro:imu_xacro xyz="0.0 0.0 0.02" />
     <xacro:laser_xacro xyz="0.0 0.0 0.10" />
     <xacro:camera_xacro xyz="0.10 0.0 0.075" />
+    <xacro:wheel_xacro wheel_name="left" xyz="0 0.10 -0.06" />
+    <xacro:wheel_xacro wheel_name="right" xyz="0 -0.10 -0.06" />
+    <xacro:caster_xacro caster_name="front" xyz="0.08 0.0 -0.076" />
+    <xacro:caster_xacro caster_name="back" xyz="-0.08 0.0 -0.076" />
 </robot>
