Commit message: 为每一个部件添加碰撞属性

File: chapt6/chapt_ws/src/fishbot_description/urdf/fishbot/actuator/caster.urdf.xacro (robot description, xacro)
@@ -12,4 +12,13 @@
                 </material>
             </visual>
+            <collision>
+                <origin xyz="0.0 0.0 0.0" rpy="0 0.0 0.0"/>
+                <geometry>
+                    <sphere radius="0.016"/>
+                </geometry>
+                <material name="yellow">
+                    <color rgba="1.0 1.0 0 0.8"/>
+                </material>
+            </collision>
         </link>
         <joint name="${caster_name}_caster_joint" type="fixed">

File: chapt6/chapt_ws/src/fishbot_description/urdf/fishbot/actuator/wheel.urdf.xacro (robot description, xacro)
@@ -12,4 +12,13 @@
                 </material>
             </visual>
+            <collision>
+                <origin xyz="0.0 0.0 0.0" rpy="1.57079 0.0 0.0"/>
+                <geometry>
+                    <cylinder radius="0.032" length="0.04"/>
+                </geometry>
+                <material name="yellow">
+                    <color rgba="1.0 1.0 0 0.8"/>
+                </material>
+            </collision>
         </link>
         <joint name="${wheel_name}_wheel_joint" type="continuous">

File: chapt6/chapt_ws/src/fishbot_description/urdf/fishbot/base.urdf.xacro (robot description, xacro)
@@ -12,4 +12,13 @@
                 </material>
             </visual>
+            <collision>
+                <origin xyz="0.0 0.0 0.0" rpy="0.0 0.0 0.0"/>
+                <geometry>
+                    <cylinder radius="${radius}" length="${length}"/>
+                </geometry>
+                <material name="white">
+                    <color rgba="1.0 1.0 1.0 0.5"/>
+                </material>
+            </collision>
         </link>
         <link name="base_footprint" />

File: chapt6/chapt_ws/src/fishbot_description/urdf/fishbot/sensor/camera.urdf.xacro (robot description, xacro)
@@ -12,4 +12,13 @@
                 </material>
             </visual>
+            <collision>
+                <origin xyz="0.0 0.0 0.0" rpy="0.0 0.0 0.0"/>
+                <geometry>
+                    <box size="0.02 0.1 0.02"/>
+                </geometry>
+                <material name="green">
+                    <color rgba="0 1.0 0 0.8"/>
+                </material>
+            </collision>
         </link>
         <joint name="camera_joint" type="fixed">

File: chapt6/chapt_ws/src/fishbot_description/urdf/fishbot/sensor/imu.urdf.xacro (robot description, xacro)
@@ -12,4 +12,13 @@
                 </material>
             </visual>
+            <collision>
+                <origin xyz="0.0 0.0 0.0" rpy="0.0 0.0 0.0"/>
+                <geometry>
+                    <box size="0.02 0.02 0.02"/>
+                </geometry>
+                <material name="black">
+                    <color rgba="0 0 0 0.8"/>
+                </material>
+            </collision>
         </link>
         <joint name="imu_joint" type="fixed">

File: chapt6/chapt_ws/src/fishbot_description/urdf/fishbot/sensor/laser.urdf.xacro (robot description, xacro)
@@ -12,4 +12,13 @@
                 </material>
             </visual>
+            <collision>
+                <origin xyz="0.0 0.0 0.0" rpy="0.0 0.0 0.0"/>
+                <geometry>
+                    <cylinder length="0.10" radius="0.01"/>
+                </geometry>
+                <material name="green">
+                    <color rgba="0 1.0 0 0.8"/>
+                </material>
+            </collision>
         </link>
         <joint name="laser_cylinder_joint" type="fixed">
@@ -28,4 +37,13 @@
                 </material>
             </visual>
+            <collision>
+                <origin xyz="0.0 0.0 0.0" rpy="0.0 0.0 0.0"/>
+                <geometry>
+                    <cylinder length="0.02" radius="0.02"/>
+                </geometry>
+                <material name="green">
+                    <color rgba="0.0 1.0 0.0 0.8"/>
+                </material>
+            </collision>
         </link>
         <joint name="laser_joint" type="fixed">

Commit message: 添加gazebo标签表示颜色，添加轮子的摩擦系数

File: chapt6/chapt_ws/src/fishbot_description/urdf/fishbot/actuator/caster.urdf.xacro (robot description, xacro)
@@ -3,4 +3,11 @@
     <xacro:include filename="$(find fishbot_description)/urdf/fishbot/common_inertia.xacro" />
     <xacro:macro name="caster_xacro" params="caster_name xyz">
+        <gazebo reference="${caster_name}_caster_link">
+            <material>Gazebo/Black</material>
+            <mu1 value="0.0" />
+            <mu2 value="0.0" />
+            <kp value="1000000000.0" />
+            <kd value="1.0" />
+        </gazebo>
         <link name="${caster_name}_caster_link">
             <visual>

File: chapt6/chapt_ws/src/fishbot_description/urdf/fishbot/actuator/wheel.urdf.xacro (robot description, xacro)
@@ -3,4 +3,11 @@
     <xacro:include filename="$(find fishbot_description)/urdf/fishbot/common_inertia.xacro" />
     <xacro:macro name="wheel_xacro" params="wheel_name xyz">
+        <gazebo reference="${wheel_name}_wheel_link">
+            <material>Gazebo/Black</material>
+            <mu1 value="20.0" />
+            <mu2 value="20.0" />
+            <kp value="1000000000.0" />
+            <kd value="1.0" />
+        </gazebo>
         <link name="${wheel_name}_wheel_link">
             <visual>

File: chapt6/chapt_ws/src/fishbot_description/urdf/fishbot/base.urdf.xacro (robot description, xacro)
@@ -3,4 +3,7 @@
     <xacro:include filename="$(find fishbot_description)/urdf/fishbot/common_inertia.xacro" />
     <xacro:macro name="base_xacro" params="length radius">
+        <gazebo reference="base_link">
+            <material>Gazebo/Yellow</material>
+        </gazebo>
         <link name="base_link">
             <visual>

File: chapt6/chapt_ws/src/fishbot_description/urdf/fishbot/sensor/camera.urdf.xacro (robot description, xacro)
@@ -3,4 +3,7 @@
     <xacro:include filename="$(find fishbot_description)/urdf/fishbot/common_inertia.xacro" />
     <xacro:macro name="camera_xacro" params="xyz">
+        <gazebo reference="camera_link">
+            <material>Gazebo/Red</material>
+        </gazebo>
         <link name="camera_link">
             <visual>

File: chapt6/chapt_ws/src/fishbot_description/urdf/fishbot/sensor/imu.urdf.xacro (robot description, xacro)
@@ -3,4 +3,7 @@
     <xacro:include filename="$(find fishbot_description)/urdf/fishbot/common_inertia.xacro" />
     <xacro:macro name="imu_xacro" params="xyz">
+        <gazebo reference="imu_link">
+            <material>Gazebo/Blue</material>
+        </gazebo>
         <link name="imu_link">
             <visual>

File: chapt6/chapt_ws/src/fishbot_description/urdf/fishbot/sensor/laser.urdf.xacro (robot description, xacro)
@@ -3,4 +3,10 @@
     <xacro:include filename="$(find fishbot_description)/urdf/fishbot/common_inertia.xacro" />
     <xacro:macro name="laser_xacro" params="xyz">
+        <gazebo reference="laser_cylinder_link">
+            <material>Gazebo/Green</material>
+        </gazebo>
+        <gazebo reference="laser_link">
+            <material>Gazebo/Black</material>
+        </gazebo>
         <link name="laser_cylinder_link">
             <visual>
