Commit message: 添加深度相机传感器仿真

File: chapt6/chapt_ws/src/fishbot_description/urdf/fishbot/plugins/gazebo_sensor_plugin.xacro (robot description, xacro)
@@ -105,4 +105,29 @@
             </sensor>
         </gazebo>
+        <gazebo reference="camera_link">
+            <sensor name="camera_sensor" type="depth">
+                <plugin name='depth_camera' filename='libgazebo_ros_camera.so'>
+                    <frame_name>camera_optical_link</frame_name>
+                </plugin>
+                <always_on>true</always_on>
+                <update_rate>10</update_rate>
+                <camera name="camera">
+                    <horizontal_fov>1.5009831567</horizontal_fov>
+                    <image>
+                        <width>800</width>
+                        <height>600</height>
+                        <format>R8G8B8</format>
+                    </image>
+                    <distortion>
+                        <k1>0.0</k1>
+                        <k2>0.0</k2>
+                        <k3>0.0</k3>
+                        <p1>0.0</p1>
+                        <p2>0.0</p2>
+                        <centor>0.5 0.5</centor>
+                    </distortion>
+                </camera>
+            </sensor>
+        </gazebo>
     </xacro:macro>
 </robot>

File: chapt6/chapt_ws/src/fishbot_description/urdf/fishbot/sensor/camera.urdf.xacro (robot description, xacro)
@@ -32,4 +32,11 @@
             <origin xyz="${xyz}"/>
         </joint>
+        <link name="camera_optical_link">
+        </link>
+        <joint name="camera_optical_joint" type="fixed">
+            <parent link="camera_link"/>
+            <child link="camera_optical_link"/>
+            <origin xyz="0 0 0" rpy="${-pi/2} 0 ${-pi/2}"/>
+        </joint>
     </xacro:macro>
 </robot>
